File: OpenEuroBoard.kicad_pcb (KiCad board)
At the start: 2 copper layers, 300 x 100 mm, 124 parts, among them J1 Eurorack_bus_mini, J10 Jack, J11 Conn_01x08, J12 Jack, J13 Jack, J14 Jack, J15 Jack, J16 Conn_01x04, J17 MIDI_in, J18 Conn_01x03, J19 Conn_01x03, J2 Conn_01x07, J20 Conn_01x03, J21 MIDI_out, J22 Conn_01x03, J23 Conn_01x05, J24 Conn_01x03, J25 Conn_01x05, J26 Conn_01x03, J27 Conn_01x08, J28 Conn_01x08, J29 Conn_01x04, J3 Conn_01x07, J30 Screw_Terminal_01x01, J31 Conn_01x05, J32 Conn_01x03, J33 Conn_01x05, J34 Conn_01x03, J35 Conn_01x05, J36 Conn_01x03, J37 Screw_Terminal_01x01, J38 Screw_Terminal_01x01, J39 Conn_01x05, J4 Conn_01x07, J40 Conn_01x03, J41 Conn_01x03, J42 Conn_01x05, J43 Conn_01x03, J44 Conn_01x03, J45 Conn_01x02, J46 Conn_01x04, J47 Screw_Terminal_01x01, J48 Screw_Terminal_01x01, J49 Screw_Terminal_01x01, J5 Conn_01x07, J50 Screw_Terminal_01x01, J51 Screw_Terminal_01x01, J52 Conn_01x04, J53 Conn_01x04, J54 Conn_01x04, J6 Jack, J7 Jack, J8 Conn_01x08, J9 Jack, SW1 SW_Push, SW10 SW_SPDT, SW11 SW_SPDT, SW12 SW_SPDT, SW2 SW_Push, SW3 SW_Push, SW4 SW_Push, SW5 SW_Push, SW6 SW_Push, SW7 SW_SPDT, SW8 SW_SPDT, SW9 SW_SPDT, U1 LM1117IMP-5, U2 TL074, U3 TL074, U4 CD40107BE, U5 6N139, U6 TL074

Commit message: Silkscreen and general rework
Parts:
- added J55: Jumpers, Connector_PinHeader_2.54mm:PinHeader_2x05_P2.54mm_Vertical, F.Cu at (234.7, 9.60)
- added J56: Conn_01x04, Connector_PinHeader_2.54mm:PinHeader_1x04_P2.54mm_Vertical, F.Cu at (245.2, 89.6)
- added J57: Conn_01x08, Connector_PinHeader_2.54mm:PinHeader_1x08_P2.54mm_Vertical, F.Cu at (297.2, 12.9)
- J10: value Jack -> Jack 4
- J12: value Jack -> Jack 5
- J13: value Jack -> Jack 6
- J14: value Jack -> Jack 7
- J15: value Jack -> Jack 8
- J6: value Jack -> Jack 1
- J7: value Jack -> Jack 2
- J9: value Jack -> Jack 3
- RV3: value 1M LOG -> 1M
- moved D3 26.5 mm to (245.5, 17.6), turned to 180 degrees
- moved D5 20.5 mm to (245.5, 25.1), turned to 180 degrees
- moved R4 19.6 mm to (232.5, 16.6), turned to 180 degrees
- moved D2 19.2 mm to (238.9, 17.6), turned to 180 degrees
- moved RV4 18.3 mm to (286.6, 80.8)
- moved SW10 18.0 mm to (213.7, 7.11)
- moved RV5 17.9 mm to (286.6, 62.9)
- moved SW9 17.7 mm to (202.7, 7.11)
- moved R5 14.6 mm to (232.5, 20.1), turned to 180 degrees
- moved J22 12.4 mm to (211.2, 20.4)
- moved D4 12.2 mm to (238.9, 25.1), turned to 180 degrees
- moved J20 12.0 mm to (200.2, 20.4)
- moved J19 11.5 mm to (211.2, 27.0)
- moved J18 11.0 mm to (200.2, 27.0)
- moved C13 9.68 mm to (276.1, 84.1)
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Other:
- board text added: "+12V +12V Test1 Test2 Test3 Test4 GND GND"
- board text added: "1"
- board text added: "2"
- board text added: "3"
- board text added: "4"
- board text added: "?"
- board text added: "CV1 GATE 1"
- board text added: "CV2 GATE 2"
- board text added: "Freq LFO 1"
- board text added: "Freq LFO 2"
- board text added: "Jack 1 Jack 2 Jack 3 Jack 4 Jack 5 Jack 6 Jack 7 Jack 8"
- board text added: "LED1 LED2 LED3 LED4"
- board text added: "MIDI IN"
- board text added: "MIDI OUT"
- board text added: "Open Eurorack Development Board https://github.com/sensai7/OpenEuroBoard"
- board text added: "SSD1306 Screen"
- board text added: "SW1"
- board text added: "SW1 SW2 SW3 SW4"
- board text added: "SW2"
- board text added: "SW3"
- board text added: "SW4"
- board text added: "Test1 Test2 Test3 Test4"
- board text removed: "Open Eurorack Development Board github.com/sensai7/xxxxx"

Commit message: Finished layout, silkscreen and routing
also fixed minijack footprint
Parts:
- added C17: 100n, Capacitor_THT:C_Disc_D3.4mm_W2.1mm_P2.50mm, F.Cu at (283.4, 16.6)
- added C18: 100n, Capacitor_THT:C_Disc_D3.4mm_W2.1mm_P2.50mm, F.Cu at (283.4, 31.8)
- added J58: Conn_01x02, Connector_PinHeader_2.54mm:PinHeader_1x02_P2.54mm_Vertical, F.Cu at (257.7, 90.1)
- added J59: AudioJack3_Ground, SensaiLib:Jack Stereo vertical Thonk, F.Cu at (284.7, 47.3)
- added TP1: TestPoint, TestPoint:TestPoint_THTPad_D3.0mm_Drill1.5mm, F.Cu at (295.8, 42.3)
- added TP2: TestPoint, TestPoint:TestPoint_THTPad_D3.0mm_Drill1.5mm, F.Cu at (295.8, 67.8)
- added TP3: TestPoint, TestPoint:TestPoint_THTPad_D3.0mm_Drill1.5mm, F.Cu at (295.8, 55.1)
- added TP4: TestPoint, TestPoint:TestPoint_THTPad_D3.0mm_Drill1.5mm, F.Cu at (295.8, 48.7)
- added TP5: TestPoint, TestPoint:TestPoint_THTPad_D3.0mm_Drill1.5mm, F.Cu at (295.8, 80.5)
- added TP6: TestPoint, TestPoint:TestPoint_THTPad_D3.0mm_Drill1.5mm, F.Cu at (295.8, 74.1)
- added TP7: TestPoint, TestPoint:TestPoint_THTPad_D3.0mm_Drill1.5mm, F.Cu at (295.8, 61.4)
- added TP8: TestPoint, TestPoint:TestPoint_THTPad_D3.0mm_Drill1.5mm, F.Cu at (295.8, 86.9)
- added U7: TL072, Package_DIP:DIP-8_W7.62mm_Socket_LongPads, F.Cu at (278.4, 20.4)
- moved R21 31.1 mm to (273.4, 71.2), turned to 180 degrees
- moved C14 26.4 mm to (252.5, 69.5), turned to 180 degrees
- moved C13 24.2 mm to (256.8, 69.5), turned to 0 degrees
- moved C12 21.6 mm to (250.0, 74.2), turned to 0 degrees
- moved C11 17.4 mm to (259.3, 74.2), turned to 180 degrees
- moved SW11 8.23 mm to (269.3, 82.8)
- moved SW12 7.91 mm to (253.9, 82.9)
- moved R15 5.77 mm to (265.7, 66.8)
- moved R20 5.75 mm to (273.3, 62.4)
- moved R17 5.72 mm to (265.7, 58.0)
- moved R16 5.70 mm to (265.7, 53.5)
- moved R14 5.67 mm to (265.7, 49.1)
- moved R18 5.65 mm to (265.7, 44.7)
- moved R19 5.62 mm to (265.7, 40.3)
- moved C15 3.53 mm to (253.3, 41.1)
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Routing:
- net +12V: track 0.00 -> 566.4 mm, vias 0 -> 1
- net -12V: track 0.00 -> 537.3 mm
- net +5V: track 0.00 -> 461.9 mm
- net Net-(J11-Pad1): track 0.00 -> 128.3 mm
- net Net-(J11-Pad2): track 0.00 -> 115.3 mm
- net TEST1: track 0.00 -> 113.1 mm
- net TEST2: track 0.00 -> 111.9 mm
- net TEST3: track 0.00 -> 108.4 mm
- net TEST4: track 0.00 -> 108.1 mm
- net Net-(J11-Pad3): track 0.00 -> 102.3 mm
- net Net-(J58-Pad1): track 0.00 -> 101.2 mm
- net SQR2: track 0.00 -> 100.3 mm, vias 0 -> 1
- net Net-(J58-Pad2): track 0.00 -> 99.6 mm
- net TRI1: track 0.00 -> 92.9 mm
- net GND: track 0.00 -> 90.2 mm, vias 0 -> 2
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- added copper zone on F.Cu, net GND
Other:
- net class power added: clearance 0.2, trace_width 0.5, via_dia 0.8, via_drill 0.4
- board text added: "+12V"
- board text added: "+5V"
- board text added: "GND"
- board text added: "L out R out"
- board text added: "Stereo Out"
- board text added: "TEST1"
- board text added: "TEST2"
- board text added: "TEST3"
- board text added: "TEST4"
- board text added: "V1.0"
- board text removed: "1/4~~250Hz"
- board text removed: "11~~11kHz"
- board text removed: "?"

Commit message: finished silkscreen, fixed some minor errors
Parts:
- added ?: , , F.Cu at (69.6, 66.8)

Commit message: stuff
Parts:
- removed ?: , 
- J10, J12, J13, J14, J15, J6, J7, J9: footprint SensaiLib:Thonkiconn Mono vertical minijack -> Connector_Audio:Jack_3.5mm_QingPu_WQP-PJ398SM_Vertical_CircularHoles
- moved J10 6.10 mm to (128.3, 3.59), turned to 0 degrees
- moved J12 6.10 mm to (143.5, 3.59), turned to 0 degrees
- moved J13 6.10 mm to (158.6, 3.59), turned to 0 degrees
- moved J14 6.10 mm to (173.8, 3.59), turned to 0 degrees
- moved J15 6.10 mm to (188.9, 3.59), turned to 0 degrees
- moved J6 6.10 mm to (82.9, 3.59), turned to 0 degrees
- moved J7 6.10 mm to (98.0, 3.59), turned to 0 degrees
- moved J9 6.10 mm to (113.2, 3.59), turned to 0 degrees
Routing:
- net Net-(R18-Pad1): track 77.4 -> 71.9 mm

Commit message: Version 1.1
Parts:
- added C19: 100n, Capacitor_THT:C_Disc_D3.4mm_W2.1mm_P2.50mm, F.Cu at (276.3, 49.8)
- added C20: 100n, Capacitor_THT:C_Disc_D3.4mm_W2.1mm_P2.50mm, F.Cu at (290.3, 40.1)
- added U8: TL074, Package_DIP:DIP-14_W7.62mm, F.Cu at (279.4, 39.4)
- R20, R21: value 100k -> 1k
- moved J59 19.1 mm to (281.6, 28.5)
- moved SW11 15.4 mm to (253.9, 83.0)
- moved SW12 15.4 mm to (269.3, 82.9)
- moved C17 13.2 mm to (283.9, 3.41)
- moved C18 13.2 mm to (283.9, 18.6)
- moved U7 13.2 mm to (278.8, 7.20)
- moved R20 10.8 mm to (263.2, 66.2), turned to 0 degrees
- moved R21 10.2 mm to (263.2, 70.4), turned to 0 degrees
- moved R15 5.37 mm to (263.1, 62.1)
- moved RV4 3.00 mm to (284.7, 85.6)
- moved RV5 3.00 mm to (284.7, 66.8)
- moved R14 2.55 mm to (263.1, 49.1)
- moved R18 2.55 mm to (263.1, 44.7)
- moved R19 2.55 mm to (263.1, 40.2)
- moved R17 2.55 mm to (263.1, 57.9)
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Connections:
- C11 pad 1: TRI1 -> TRI1PRE
- C12 pad 1: TRI2 -> TRI2PRE
- C12 pad 2: Net-(C12-Pad2) -> Net-(U8D--)
- C14 pad 1: Net-(C12-Pad2) -> Net-(U8D--)
- J10 pad TN: Net-(J10-PadTN) -> unconnected-(J10-PadTN)
- J12 pad TN: Net-(J12-PadTN) -> unconnected-(J12-PadTN)
- J13 pad TN: Net-(J13-PadTN) -> unconnected-(J13-PadTN)
- J14 pad TN: Net-(J14-PadTN) -> unconnected-(J14-PadTN)
- J15 pad TN: Net-(J15-PadTN) -> unconnected-(J15-PadTN)
- J17 pad 1: Net-(J17-Pad1) -> unconnected-(J17-Pad1)
- J17 pad 2: Net-(J17-Pad2) -> unconnected-(J17-Pad2)
- J17 pad 3: Net-(J17-Pad3) -> unconnected-(J17-Pad3)
- J21 pad 1: Net-(J21-Pad1) -> unconnected-(J21-Pad1)
- J21 pad 2: Net-(J21-Pad2) -> unconnected-(J21-Pad2)
- J21 pad 3: Net-(J21-Pad3) -> unconnected-(J21-Pad3)
- J30 pad 1: Net-(J30-Pad1) -> unconnected-(J30-Pin_1-Pad1)
- J37 pad 1: Net-(J37-Pad1) -> unconnected-(J37-Pin_1-Pad1)
- J38 pad 1: Net-(J38-Pad1) -> unconnected-(J38-Pin_1-Pad1)
- J47 pad 1: Net-(J47-Pad1) -> unconnected-(J47-Pin_1-Pad1)
- J48 pad 1: Net-(J48-Pad1) -> unconnected-(J48-Pin_1-Pad1)
- J49 pad 1: Net-(J49-Pad1) -> unconnected-(J49-Pin_1-Pad1)
- J50 pad 1: Net-(J50-Pad1) -> unconnected-(J50-Pin_1-Pad1)
- J51 pad 1: Net-(J51-Pad1) -> unconnected-(J51-Pin_1-Pad1)
- J55 pad 1: Net-(J55-Pad1) -> unconnected-(J55-Pin_1-Pad1)
- J55 pad 10: Net-(J55-Pad10) -> unconnected-(J55-Pin_10-Pad10)
- J55 pad 2: Net-(J55-Pad2) -> unconnected-(J55-Pin_2-Pad2)
- J55 pad 3: Net-(J55-Pad3) -> unconnected-(J55-Pin_3-Pad3)
- J55 pad 4: Net-(J55-Pad4) -> unconnected-(J55-Pin_4-Pad4)
- J55 pad 5: Net-(J55-Pad5) -> unconnected-(J55-Pin_5-Pad5)
- J55 pad 6: Net-(J55-Pad6) -> unconnected-(J55-Pin_6-Pad6)
- J55 pad 7: Net-(J55-Pad7) -> unconnected-(J55-Pin_7-Pad7)
- J55 pad 8: Net-(J55-Pad8) -> unconnected-(J55-Pin_8-Pad8)
- J55 pad 9: Net-(J55-Pad9) -> unconnected-(J55-Pin_9-Pad9)
- J59 pad G: Net-(J59-PadG) -> unconnected-(J59-PadG)
- J6 pad TN: Net-(J6-PadTN) -> unconnected-(J6-PadTN)
- J7 pad TN: Net-(J7-PadTN) -> unconnected-(J7-PadTN)
- J9 pad TN: Net-(J9-PadTN) -> unconnected-(J9-PadTN)
- R14 pad 1: TRI1 -> TRI1PRE
- R15 pad 1: TRI2 -> TRI2PRE
- R15 pad 2: Net-(R15-Pad2) -> Net-(U8C-+)
- R16 pad 1: SQR1 -> SQR1PRE
- R17 pad 1: SQR2 -> SQR2PRE
- R17 pad 2: Net-(R15-Pad2) -> Net-(U8C-+)
- R18 pad 2: SQR1 -> SQR1PRE
- R19 pad 2: SQR2 -> SQR2PRE
- R20 pad 1: GND -> Net-(R20-Pad1)
- R20 pad 2: Net-(R20-Pad2) -> SQR1PRE
- R21 pad 1: GND -> SQR2PRE
- RV1 pad 1: +5V -> GND
- RV1 pad 3: GND -> +5V
- RV2 pad 1: +5V -> GND
- RV2 pad 3: GND -> +5V
- RV5 pad 3: Net-(C12-Pad2) -> Net-(U8D--)
- SW11 pad 1: TRI1 -> TRI1PRE
- SW11 pad 3: Net-(R20-Pad2) -> unconnected-(SW11-C-Pad3)
- SW12 pad 1: TRI2 -> TRI2PRE
- SW12 pad 3: Net-(R21-Pad2) -> unconnected-(SW12-C-Pad3)
- U5 pad 1: Net-(U5-Pad1) -> unconnected-(U5-NC-Pad1)
- U5 pad 4: Net-(U5-Pad4) -> unconnected-(U5-NC-Pad4)
- U5 pad 7: Net-(U5-Pad7) -> unconnected-(U5-VO1-Pad7)
- U6 pad 1: SQR2 -> SQR1
- U6 pad 14: TRI1 -> TRI1PRE
- U6 pad 2: GND -> SQR1
- U6 pad 3: Net-(R15-Pad2) -> SQR1PRE
- U6 pad 5: GND -> TRI1PRE
- U6 pad 6: Net-(C12-Pad2) -> TRI1
- U6 pad 7: TRI2 -> TRI1
- U6 pad 8: SQR1 -> Net-(R20-Pad1)
Routing:
- net GND: track 90.2 -> 810.6 mm, vias 2 -> 0
- net TRI2PRE: track 0.00 -> 96.8 mm
- net Net-(U8D--): track 0.00 -> 84.2 mm
- net TRI1PRE: track 0.00 -> 67.7 mm
- net TRI1: track 92.9 -> 27.5 mm
- net Net-(C12-Pad2): track 59.2 -> 0.00 mm, vias 2 -> 0
- net +12V: track 566.4 -> 512.6 mm
- net SQR1PRE: track 0.00 -> 47.8 mm
- net SQR2PRE: track 0.00 -> 46.1 mm, vias 0 -> 1
- net Net-(R15-Pad2): track 38.6 -> 0.00 mm, vias 1 -> 0
- net -12V: track 537.3 -> 501.9 mm, vias 0 -> 1
- net SQR2: track 100.3 -> 70.7 mm
- net SQR1: track 69.1 -> 44.2 mm, vias 1 -> 0
- net Net-(U7B--): track 30.7 -> 54.7 mm
- net Net-(U8C-+): track 0.00 -> 24.0 mm
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- added copper zone on B.Cu, net GND
Other:
- net class Default removed
- net class power removed
- board text added: "Jack 1"
- board text added: "Jack 2"
- board text added: "Jack 3"
- board text added: "Jack 4"
- board text added: "Jack 5"
- board text added: "Jack 6"
- board text added: "Jack 7"
- board text added: "Jack 8"
- board text added: "L H"
- board text added: "Open Eurorack Development Board v1.1 https://github.com/sensai7/OpenEuroBoard"
- board text removed: "Open Eurorack Development Board https://github.com/sensai7/OpenEuroBoard"
